File: hardware/ms/ms.kicad_pcb (KiCad board)
At the start: 2 copper layers, 13 parts

Commit message: sch finished
Parts:
- removed REF** (x13): LED, Library:LED
- added C1: 33p, Capacitor_SMD:C_0603_1608Metric, F.Cu at (144.7, 122.6)
- added C10: 100n, Capacitor_SMD:C_0603_1608Metric, F.Cu at (144.7, 145.2)
- added C11: 100n, Capacitor_SMD:C_0603_1608Metric, F.Cu at (148.7, 122.6)
- added C12: 100n, Capacitor_SMD:C_0603_1608Metric, F.Cu at (148.7, 125.1)
- added C13: 10u, Capacitor_SMD:C_0603_1608Metric, F.Cu at (148.7, 127.6)
- added C14: 100n, Capacitor_SMD:C_0603_1608Metric, F.Cu at (148.7, 130.1)
- added C15: 10u, Capacitor_SMD:C_0603_1608Metric, F.Cu at (148.7, 132.6)
- added C16: 100n, Capacitor_SMD:C_0603_1608Metric, F.Cu at (148.7, 135.1)
- added C17: 1u, Capacitor_SMD:C_0603_1608Metric, F.Cu at (148.7, 137.6)
- added C18: 1u, Capacitor_SMD:C_0603_1608Metric, F.Cu at (148.7, 140.2)
- added C19: 4u7, Capacitor_SMD:C_0603_1608Metric, F.Cu at (148.7, 142.7)
- added C2: 33p, Capacitor_SMD:C_0603_1608Metric, F.Cu at (144.7, 125.1)
- added C20: 100n, Capacitor_SMD:C_0603_1608Metric, F.Cu at (148.7, 145.2)
- added C21: 4u7, Capacitor_SMD:C_0603_1608Metric, F.Cu at (152.7, 122.6)
- added C22: 100n, Capacitor_SMD:C_0603_1608Metric, F.Cu at (152.7, 125.1)
- added C23: 2u2, Capacitor_SMD:C_0603_1608Metric, F.Cu at (152.7, 127.6)
- added C24: 4u7, Capacitor_SMD:C_0603_1608Metric, F.Cu at (152.7, 130.1)
- added C3: 100n, Capacitor_SMD:C_0603_1608Metric, F.Cu at (144.7, 127.6)
- added C4: 33p, Capacitor_SMD:C_0603_1608Metric, F.Cu at (144.7, 130.1)
- added C5: 33p, Capacitor_SMD:C_0603_1608Metric, F.Cu at (144.7, 132.6)
- added C6: 100n, Capacitor_SMD:C_0603_1608Metric, F.Cu at (144.7, 135.1)
- added C7: 10u, Capacitor_SMD:C_0603_1608Metric, F.Cu at (144.7, 137.6)
- added C8: 10u, Capacitor_SMD:C_0603_1608Metric, F.Cu at (144.7, 140.2)
- added C9: 100n, Capacitor_SMD:C_0603_1608Metric, F.Cu at (144.7, 142.7)
- added D1: LED, Capacitor_SMD:C_0603_1608Metric, F.Cu at (152.7, 132.6)
- added D10: LED, LED_THT:LED_D5.0mm_Clear, F.Cu at (100.3, 143.1)
- added D11: LED, LED_THT:LED_D5.0mm_Clear, F.Cu at (107.8, 83.3)
- added D12: LED, LED_THT:LED_D5.0mm_Clear, F.Cu at (107.8, 90.8)
- added D13: LED, LED_THT:LED_D5.0mm_Clear, F.Cu at (107.8, 98.3)
- added D14: LED, LED_THT:LED_D5.0mm_Clear, F.Cu at (107.8, 105.8)
- added D15: LED, LED_THT:LED_D5.0mm_Clear, F.Cu at (107.8, 113.2)
- added D16: LED, LED_THT:LED_D5.0mm_Clear, F.Cu at (107.8, 120.7)
- added D17: LED, LED_THT:LED_D5.0mm_Clear, F.Cu at (107.8, 128.2)
- added D18: LED, LED_THT:LED_D5.0mm_Clear, F.Cu at (107.8, 135.6)
- added D19: LED, LED_THT:LED_D5.0mm_Clear, F.Cu at (107.8, 143.1)
- added D2: LED, LED_THT:LED_D5.0mm_Clear, F.Cu at (100.3, 83.3)
- added D20: LED, LED_THT:LED_D5.0mm_Clear, F.Cu at (115.3, 83.3)
- added D21: LED, LED_THT:LED_D5.0mm_Clear, F.Cu at (115.3, 90.8)
- added D22: LED, LED_THT:LED_D5.0mm_Clear, F.Cu at (115.3, 98.3)
- added D23: LED, LED_THT:LED_D5.0mm_Clear, F.Cu at (115.3, 105.8)
- added D24: LED, LED_THT:LED_D5.0mm_Clear, F.Cu at (115.3, 113.2)
- added D25: LED, LED_THT:LED_D5.0mm_Clear, F.Cu at (115.3, 120.7)
- added D26: LED, LED_THT:LED_D5.0mm_Clear, F.Cu at (115.3, 128.2)
- added D27: LED, LED_THT:LED_D5.0mm_Clear, F.Cu at (115.3, 135.6)
- added D28: LED, LED_THT:LED_D5.0mm_Clear, F.Cu at (115.3, 143.1)
- added D29: LED, LED_THT:LED_D5.0mm_Clear, F.Cu at (122.7, 83.3)
- added D3: LED, LED_THT:LED_D5.0mm_Clear, F.Cu at (100.3, 90.8)
- added D30: LED, LED_THT:LED_D5.0mm_Clear, F.Cu at (122.7, 90.8)
- added D31: LED, LED_THT:LED_D5.0mm_Clear, F.Cu at (122.7, 98.3)
- added D32: LED, LED_THT:LED_D5.0mm_Clear, F.Cu at (122.7, 105.8)
- added D33: LED, LED_THT:LED_D5.0mm_Clear, F.Cu at (122.7, 113.2)
- added D34: LED, LED_THT:LED_D5.0mm_Clear, F.Cu at (122.7, 120.7)
- added D35: LED, LED_THT:LED_D5.0mm_Clear, F.Cu at (122.7, 128.2)
- added D36: LED, LED_THT:LED_D5.0mm_Clear, F.Cu at (122.7, 135.6)
- added D37: LED, LED_THT:LED_D5.0mm_Clear, F.Cu at (122.7, 143.1)
- added D38: LED, LED_THT:LED_D5.0mm_Clear, F.Cu at (130.2, 83.3)
- added D39: LED, LED_THT:LED_D5.0mm_Clear, F.Cu at (130.2, 90.8)
- added D4: LED, LED_THT:LED_D5.0mm_Clear, F.Cu at (100.3, 98.3)
- added D40: LED, LED_THT:LED_D5.0mm_Clear, F.Cu at (130.2, 98.3)
- added D41: LED, LED_THT:LED_D5.0mm_Clear, F.Cu at (130.2, 105.8)
- added D42: LED, LED_THT:LED_D5.0mm_Clear, F.Cu at (130.2, 113.2)
- added D43: LED, LED_THT:LED_D5.0mm_Clear, F.Cu at (130.2, 120.7)
- added D44: LED, LED_THT:LED_D5.0mm_Clear, F.Cu at (130.2, 128.2)
- added D45: LED, LED_THT:LED_D5.0mm_Clear, F.Cu at (130.2, 135.6)
- added D46: LED, LED_THT:LED_D5.0mm_Clear, F.Cu at (130.2, 143.1)
- added D47: LED, LED_THT:LED_D5.0mm_Clear, F.Cu at (137.7, 83.3)
- added D48: LED, LED_THT:LED_D5.0mm_Clear, F.Cu at (137.7, 90.8)
- added D49: LED, LED_THT:LED_D5.0mm_Clear, F.Cu at (137.7, 98.3)
- added D5: LED, LED_THT:LED_D5.0mm_Clear, F.Cu at (100.3, 105.8)
- added D50: LED, LED_THT:LED_D5.0mm_Clear, F.Cu at (137.7, 105.8)
- added D51: LED, LED_THT:LED_D5.0mm_Clear, F.Cu at (137.7, 113.2)
- added D52: LED, LED_THT:LED_D5.0mm_Clear, F.Cu at (137.7, 120.7)
- added D53: 3v3, Diode_SMD:D_SOD-123, F.Cu at (164.5, 101.0)
- added D54: 3v3, Diode_SMD:D_SOD-123, F.Cu at (164.5, 104.4)
- added D55: 3v3, Diode_SMD:D_SOD-123, F.Cu at (164.5, 107.7)
- added D56: 3v3, Diode_SMD:D_SOD-123, F.Cu at (164.5, 111.1)
- added D57: LED, LED_SMD:LED_0805_2012Metric, F.Cu at (150.1, 147.9)
- added D58: LED, Capacitor_SMD:C_0603_1608Metric, F.Cu at (152.7, 135.1)
- added D59: LED, Capacitor_SMD:C_0603_1608Metric, F.Cu at (152.7, 137.6)
- added D6: LED, LED_THT:LED_D5.0mm_Clear, F.Cu at (100.3, 113.2)
- added D60: LED, Capacitor_SMD:C_0603_1608Metric, F.Cu at (152.7, 140.2)
- added D61: LED, Capacitor_SMD:C_0603_1608Metric, F.Cu at (152.7, 142.7)
- added D7: LED, LED_THT:LED_D5.0mm_Clear, F.Cu at (100.3, 120.7)
- added D8: LED, LED_THT:LED_D5.0mm_Clear, F.Cu at (100.3, 128.2)
- added D9: LED, LED_THT:LED_D5.0mm_Clear, F.Cu at (100.3, 135.6)
- added DS1: OLED-128O032D, Library:OLED-128O032D, F.Cu at (147.9, 119.6)
- added J1: DBG, Connector_PinHeader_2.54mm:PinHeader_1x08_P2.54mm_Vertical, F.Cu at (169.1, 123.6)
- added J2: BAT, Connector_JST:JST_XH_B2B-XH-A_1x02_P2.50mm_Vertical, F.Cu at (165.1, 116.1)
- added R1: 470k, Resistor_SMD:R_0603_1608Metric, F.Cu at (152.7, 145.2)
- added R10: 0, Resistor_SMD:R_0603_1608Metric, F.Cu at (156.8, 142.7)
- added R11: 470k, Resistor_SMD:R_0603_1608Metric, F.Cu at (156.8, 145.2)
- added R12: 1k, Resistor_SMD:R_0603_1608Metric, F.Cu at (160.8, 122.6)
- added R13: 100k, Resistor_SMD:R_0603_1608Metric, F.Cu at (160.8, 125.1)
- added R14: 100k, Resistor_SMD:R_0603_1608Metric, F.Cu at (160.8, 127.6)
- added R15: 100k, Resistor_SMD:R_0603_1608Metric, F.Cu at (160.8, 130.1)
- added R16: 100k, Resistor_SMD:R_0603_1608Metric, F.Cu at (160.8, 132.6)
- added R17: 100k, Resistor_SMD:R_0603_1608Metric, F.Cu at (160.8, 135.1)
- added R18: 100k, Resistor_SMD:R_0603_1608Metric, F.Cu at (160.8, 137.6)
- added R19: NC, Resistor_SMD:R_0603_1608Metric, F.Cu at (160.8, 140.2)
- added R2: 0, Resistor_SMD:R_0603_1608Metric, F.Cu at (156.8, 122.6)
- added R20: 100k, Resistor_SMD:R_0603_1608Metric, F.Cu at (160.8, 142.7)
- added R21: 1M, Resistor_SMD:R_0603_1608Metric, F.Cu at (160.8, 145.2)
- added R22: 1M, Resistor_SMD:R_0603_1608Metric, F.Cu at (164.8, 122.6)
- added R23: 10k, Resistor_SMD:R_0603_1608Metric, F.Cu at (164.8, 125.1)
- added R24: 10k, Resistor_SMD:R_0603_1608Metric, F.Cu at (164.8, 127.6)
- added R25: 10k, Resistor_SMD:R_0603_1608Metric, F.Cu at (164.8, 130.1)
- added R26: 560k, Resistor_SMD:R_0603_1608Metric, F.Cu at (164.8, 132.6)
- added R27: 4k7, Resistor_SMD:R_0603_1608Metric, F.Cu at (164.8, 135.1)
- added R28: 4k7, Resistor_SMD:R_0603_1608Metric, F.Cu at (164.8, 137.6)
- added R29: 4k7, Resistor_SMD:R_0603_1608Metric, F.Cu at (164.8, 140.2)
- added R3: 1k, Resistor_SMD:R_0603_1608Metric, F.Cu at (156.8, 125.1)
- added R4: 0, Resistor_SMD:R_0603_1608Metric, F.Cu at (156.8, 127.6)
- added R5: 470k, Resistor_SMD:R_0603_1608Metric, F.Cu at (156.8, 130.1)
- added R6: 1k, Resistor_SMD:R_0603_1608Metric, F.Cu at (156.8, 132.6)
- added R7: 0, Resistor_SMD:R_0603_1608Metric, F.Cu at (156.8, 135.1)
- added R8: 470k, Resistor_SMD:R_0603_1608Metric, F.Cu at (156.8, 137.6)
- added R9: 1k, Resistor_SMD:R_0603_1608Metric, F.Cu at (156.8, 140.2)
- added RV1: 2k, Potentiometer_SMD:Potentiometer_Bourns_TC33X_Vertical, F.Cu at (158.6, 101.7)
- added RV2: 2k, Potentiometer_SMD:Potentiometer_Bourns_TC33X_Vertical, F.Cu at (158.6, 106.5)
- added RV3: 2k, Potentiometer_SMD:Potentiometer_Bourns_TC33X_Vertical, F.Cu at (158.6, 111.2)
- added RV4: 2k, Potentiometer_SMD:Potentiometer_Bourns_TC33X_Vertical, F.Cu at (158.6, 116.0)
- added SW1: BUTTON, Button_Switch_SMD:SW_Push_1P1T_NO_Vertical_Wuerth_434133025816, F.Cu at (167.3, 82.0)
- added SW2: RESET, Button_Switch_SMD:SW_Push_1P1T_NO_Vertical_Wuerth_434133025816, F.Cu at (167.3, 86.7)
- added U1: TLV75733PDBV, Package_TO_SOT_SMD:SOT-23-5, F.Cu at (145.3, 148.8)
- added U2: STM32G031G8Ux, Package_DFN_QFN:QFN-28_4x4mm_P0.5mm, F.Cu at (167.4, 92.3)
- added U3: OP_T, Package_SO:SOIC-8_3.9x4.9mm_P1.27mm, F.Cu at (159.7, 83.0)
- added U4: OP_B, Package_SO:SOIC-8_3.9x4.9mm_P1.27mm, F.Cu at (159.7, 89.5)
- added U5: Opamp_Dual, Package_SO:SOIC-8_3.9x4.9mm_P1.27mm, F.Cu at (159.7, 96.1)

Commit message: hw pcb init
Parts:
- removed the D1 at (152.7, 132.6)
- removed the D10 at (100.3, 143.1)
- removed the D14 at (107.8, 105.8)
- removed the D15 at (107.8, 113.2)
- removed the D16 at (107.8, 120.7)
- removed the D19 at (107.8, 143.1)
- removed the D2 at (100.3, 83.3)
- removed the D23 at (115.3, 105.8)
- removed the D27 at (115.3, 135.6)
- removed the D28 at (115.3, 143.1)
- removed the D29 at (122.7, 83.3)
- removed the D3 at (100.3, 90.8)
- removed the D32 at (122.7, 105.8)
- removed the D40 at (130.2, 98.3)
- removed the D41 at (130.2, 105.8)
- removed D42, D45, D49: LED, LED_THT:LED_D5.0mm_Clear
- removed D59, D60, D61: LED, Capacitor_SMD:C_0603_1608Metric
- removed the D6 at (100.3, 113.2)
- added D34: LED, LED_THT:LED_D5.0mm_Clear, F.Cu at (178.3, 76.9)
- added D35: LED, LED_THT:LED_D5.0mm_Clear, F.Cu at (178.3, 132.8)
- added H1: MountingHole_Pad, MountingHole:MountingHole_3.2mm_M3_Pad, F.Cu at (169.4, 123.8)
- added H2: MountingHole_Pad, MountingHole:MountingHole_3.2mm_M3_Pad, F.Cu at (131.4, 85.8)
- added H3: MountingHole_Pad, MountingHole:MountingHole_3.2mm_M3_Pad, F.Cu at (169.4, 85.8)
- added H4: MountingHole_Pad, MountingHole:MountingHole_3.2mm_M3_Pad, F.Cu at (131.4, 123.8)
- D33: renamed from D58; footprint Capacitor_SMD:C_0603_1608Metric -> LED_THT:LED_D5.0mm_Clear
- DS1: moved to B.Cu
- moved C14 104.9 mm to (66.5, 64.9)
- moved R25 104.9 mm to (82.6, 64.9)
- moved C11 104.9 mm to (66.5, 57.4)
- moved C12 104.9 mm to (66.5, 59.9)
- moved C13 104.9 mm to (66.5, 62.4)
- moved C15 104.9 mm to (66.5, 67.4)
- moved C16 104.9 mm to (66.5, 69.9)
- moved C17 104.9 mm to (66.5, 72.4)
- moved C18 104.9 mm to (66.5, 75.0)
- moved C19 104.9 mm to (66.5, 77.5)
- moved C20 104.9 mm to (66.5, 80.0)
- moved C22 104.9 mm to (70.5, 59.9)
- moved C24 104.9 mm to (70.5, 64.9)
- moved R10 104.9 mm to (74.5, 77.5)
- moved R22 104.9 mm to (82.6, 57.4)
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- renumbered D4 to D1, D17 to D10, D26 to D14, D22 to D15, D18 to D16, D44 to D17, D48 to D18, D52 to D19, D5 to D2, D39 to D20, D35 to D21, D31 to D22, D43 to D23, D47 to D24, D51 to D25, D38 to D26, D34 to D27, D30 to D28, D46 to D29, D24 to D3, D50 to D30, D37 to D31, D33 to D32, D53 to D37, D54 to D38, D55 to D39, D20 to D4, D56 to D40, D57 to D41, D7 to D5, D8 to D6, D9 to D7, D25 to D8, D21 to D9
Connections:
- D36 pad 1: /ARR_BR -> GND
- D36 pad 2: GND -> Net-(D36-A)
- R10 pad 2: Net-(U4B--) -> Net-(U4A-+)
- R7 pad 2: Net-(U4A-+) -> Net-(U4B--)
- RV4 pad 3: Net-(D61-A) -> Net-(D36-A)
- U4 pad 1: Net-(C4-Pad2) -> Net-(C5-Pad2)
- U4 pad 2: /ARR_BL -> /ARR_BR
- U4 pad 5: /ARR_BR -> /ARR_BL
- U4 pad 7: Net-(C5-Pad2) -> Net-(C4-Pad2)
Other:
- board outline added: 60 x 60 mm

Commit message: hw ver1
Parts:
- added C25: 10u, Capacitor_SMD:C_0603_1608Metric, F.Cu at (125.1, 103.2)
- added C26: 10u, Capacitor_SMD:C_0603_1608Metric, F.Cu at (132.0, 105.2)
- added C27: 100n, Capacitor_SMD:C_0603_1608Metric, F.Cu at (133.4, 105.2)
- added G***: LOGO, LOGO, F.Cu at (172.7, 113.6)
- added J3: USB_C_Receptacle_PowerOnly_6P, Connector_USB:USB_C_Receptacle_GCT_USB4125-xx-x_6P_TopMnt_Horizontal, F.Cu at (123.9, 93.0)
- added R30: 5k1, Resistor_SMD:R_0603_1608Metric, F.Cu at (129.0, 90.5)
- added R31: 5k1, Resistor_SMD:R_0603_1608Metric, F.Cu at (129.0, 93.5)
- added R32: 5k1, Resistor_SMD:R_0603_1608Metric, F.Cu at (125.1, 100.2)
- added U6: TP4056-42-ESOP8, Package_SO:SOIC-8-1EP_3.9x4.9mm_P1.27mm_EP2.41x3.3mm, F.Cu at (130.6, 101.0)
- moved C17 116.2 mm to (178.8, 102.5), turned to 90 degrees
- moved C21 114.4 mm to (175.7, 102.5), turned to -90 degrees
- moved C18 114.2 mm to (177.3, 102.5), turned to 90 degrees
- moved C15 113.5 mm to (164.1, 125.5)
- moved C16 113.1 mm to (164.1, 127.0)
- moved C22 112.1 mm to (174.2, 102.5), turned to -90 degrees
- moved D40 109.8 mm to (160.0, 123.5), turned to 90 degrees
- moved C5 109.5 mm to (156.5, 123.5), turned to -90 degrees
- moved C23 108.4 mm to (171.2, 102.5), turned to -90 degrees
- moved C13 107.6 mm to (151.3, 128.7), turned to 180 degrees
- moved C14 107.0 mm to (151.3, 130.2), turned to 180 degrees
- moved C24 107.0 mm to (171.7, 99.8), turned to 180 degrees
- moved C19 106.2 mm to (169.7, 102.5), turned to -90 degrees
- moved R12 104.5 mm to (157.3, 126.0), turned to 180 degrees
- moved C6 104.3 mm to (148.9, 128.3), turned to -90 degrees
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Connections:
- C1 pad 2: Net-(C1-Pad2) -> /O1
- C2 pad 2: Net-(C2-Pad2) -> /O2
- C4 pad 2: Net-(C4-Pad2) -> /O3
- C5 pad 2: Net-(C5-Pad2) -> /O4
- J1 pad 3: /SWCLK -> GND
- J1 pad 5: /U1TXD -> /SWCLK
- J1 pad 6: /U1RXD -> /U1TXD
- J1 pad 7: /~{RESET} -> /U1RXD
- J1 pad 8: GND -> /~{RESET}
- R1 pad 2: Net-(C1-Pad2) -> /O1
- R11 pad 2: Net-(C5-Pad2) -> /O4
- R12 pad 2: Net-(C5-Pad2) -> /O4
- R15 pad 1: /ARR_BR -> /O4
- R16 pad 1: /ARR_BL -> /O3
- R17 pad 1: /ARR_TR -> /O2
- R18 pad 1: /ARR_TL -> /O1
- R3 pad 2: Net-(C1-Pad2) -> /O1
- R4 pad 2: Net-(U3B--) -> Net-(U3B-+)
- R5 pad 2: Net-(C2-Pad2) -> /O2
- R6 pad 2: Net-(C2-Pad2) -> /O2
- R7 pad 2: Net-(U4B--) -> Net-(U4B-+)
- R8 pad 2: Net-(C4-Pad2) -> /O3
- R9 pad 2: Net-(C4-Pad2) -> /O3
- U3 pad 1: Net-(C1-Pad2) -> /O1
- U3 pad 5: /ARR_TR -> Net-(U3B-+)
- U3 pad 6: Net-(U3B--) -> /ARR_TR
- U3 pad 7: Net-(C2-Pad2) -> /O2
- U4 pad 1: Net-(C5-Pad2) -> /O4
- U4 pad 5: /ARR_BL -> Net-(U4B-+)
- U4 pad 6: Net-(U4B--) -> /ARR_BL
- U4 pad 7: Net-(C4-Pad2) -> /O3
Routing:
- net +3V3: track 0.00 -> 203.2 mm, vias 0 -> 7
- net VCC: track 0.00 -> 102.6 mm, vias 0 -> 4
- net /~{RES}: track 0.00 -> 83.8 mm, vias 0 -> 2
- net /O4: track 0.00 -> 65.2 mm, vias 0 -> 2
- net /O3: track 0.00 -> 63.3 mm
- net /SDA: track 0.00 -> 54.3 mm, vias 0 -> 5
- net /SCL: track 0.00 -> 53.8 mm, vias 0 -> 3
- net /~{RESET}: track 0.00 -> 52.8 mm, vias 0 -> 3
- net /ARR_BR: track 0.00 -> 52.5 mm
- net /ARR_TL: track 0.00 -> 51.7 mm
- net /ARR_TR: track 0.00 -> 48.8 mm
- net /ARR_BL: track 0.00 -> 48.7 mm
- net /BUTTON: track 0.00 -> 37.4 mm, vias 0 -> 2
- net /SWCLK: track 0.00 -> 35.5 mm, vias 0 -> 1
- net /SWDIO: track 0.00 -> 35.4 mm, vias 0 -> 1
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- added copper zone on B.Cu, net GND
- added copper zone on F.Cu, net GND
Other:
- board text added: "JLCJLCJLCJLC"

Commit message: hw rev2
Parts:
- added R33: 10k, Resistor_SMD:R_0603_1608Metric, F.Cu at (132.0, 93.5)
- added R34: 10k, Resistor_SMD:R_0603_1608Metric, F.Cu at (131.2, 95.8)
Connections:
- U2 pad 6: /ADC_IN0 -> Net-(U2-PA0)
Routing:
- net /ADC_IN0: track 35.0 -> 18.4 mm, vias 2 -> 1
- net Net-(U2-PA0): track 0.00 -> 15.7 mm, vias 0 -> 2
- net GND: track 12.2 -> 13.5 mm, vias 158 -> 170
