File: hardware/ms/ms.kicad_sch (KiCad schematic)
At the start: 4 parts, among them U1 TP4056-42-ESOP8, U2 STM32G031G8Ux, U3 Opamp_Dual

Commit message: hardware update
Parts:
- added D10, D100, D101, D102, D103, D104, D105, D106, D107, D108, D109, D11, D110, D111, D112, D113, D114, D115, D116, D117, D118, D119, D12, D120, D121, D122, D123, D124, D125, D126, D127, D128, D129, D13, D130, D131, D132, D133, D134, D135, D136, D137, D138, D139, D14, D140, D141, D142, D143, D144, D145, D146, D147, D148, D149, D15, D150, D151, D152, D153, D154, D155, D156, D157, D158, D159, D16, D160, D161, D162, D163, D164, D165, D166, D167, D168, D169, D17, D170, D171, D172, D173, D174, D175, D176, D177, D178, D179, D18, D180, D181, D182, D183, D184, D185, D186, D187, D188, D189, D19, D190, D191, D192, D193, D194, D195, D196, D197, D198, D199, D2, D20, D200, D21, D22, D23, D24, D25, D26, D27, D28, D29, D3, D30, D31, D32, D33, D34, D35, D36, D37, D38, D39, D4, D40, D41, D42, D43, D44, D45, D46, D47, D48, D49, D5, D50, D51, D52, D53, D54, D55, D56, D57, D58, D59, D6, D60, D61, D62, D63, D64, D65, D66, D67, D68, D69, D7, D70, D71, D72, D73, D74, D75, D76, D77, D78, D79, D8, D80, D81, D82, D83, D84, D85, D86, D87, D88, D89, D9, D90, D91, D92, D93, D94, D95, D96, D97, D98, D99: LED, Library:LED, symbol Device:LED
Connections:
- net GND: now reaches D1.2 (A)
- net GND: now also D10.2 (A), D100.2 (A), D101.2 (A), D102.2 (A), D103.2 (A), D104.2 (A), D105.2 (A), D106.2 (A), D107.2 (A), D108.2 (A), D109.2 (A), D11.2 (A), D110.2 (A), D111.2 (A), D112.2 (A), D113.2 (A), D114.2 (A), D115.2 (A), D116.2 (A), D117.2 (A), D118.2 (A), D119.2 (A), D12.2 (A), D120.2 (A), D121.2 (A), D122.2 (A), D123.2 (A), D124.2 (A), D125.2 (A), D126.2 (A), D127.2 (A), D128.2 (A), D129.2 (A), D13.2 (A), D130.2 (A), D131.2 (A), D132.2 (A), D133.2 (A), D134.2 (A), D135.2 (A), D136.2 (A), D137.2 (A), D138.2 (A), D139.2 (A), D14.2 (A), D140.2 (A), D141.2 (A), D142.2 (A), D143.2 (A), D144.2 (A), D145.2 (A), D146.2 (A), D147.2 (A), D148.2 (A), D149.2 (A), D15.2 (A), D150.2 (A), D151.2 (A), D152.2 (A), D153.2 (A), D154.2 (A), D155.2 (A), D156.2 (A), D157.2 (A), D158.2 (A), D159.2 (A), D16.2 (A), D160.2 (A), D161.2 (A), D162.2 (A), D163.2 (A), D164.2 (A), D165.2 (A), D166.2 (A), D167.2 (A), D168.2 (A), D169.2 (A), D17.2 (A), D170.2 (A), D171.2 (A), D172.2 (A), D173.2 (A), D174.2 (A), D175.2 (A), D176.2 (A), D177.2 (A), D178.2 (A), D179.2 (A), D18.2 (A), D180.2 (A), D181.2 (A), D182.2 (A), D183.2 (A), D184.2 (A), D185.2 (A), D186.2 (A), D187.2 (A), D188.2 (A), D189.2 (A), D19.2 (A), D190.2 (A), D191.2 (A), D192.2 (A), D193.2 (A), D194.2 (A), D195.2 (A), D196.2 (A), D197.2 (A), D198.2 (A), D199.2 (A), D2.2 (A), D20.2 (A), D200.2 (A), D21.2 (A), D22.2 (A), D23.2 (A), D24.2 (A), D25.2 (A), D26.2 (A), D27.2 (A), D28.2 (A), D29.2 (A), D3.2 (A), D30.2 (A), D31.2 (A), D32.2 (A), D33.2 (A), D34.2 (A), D35.2 (A), D36.2 (A), D37.2 (A), D38.2 (A), D39.2 (A), D4.2 (A), D40.2 (A), D41.2 (A), D42.2 (A), D43.2 (A), D44.2 (A), D45.2 (A), D46.2 (A), D47.2 (A), D48.2 (A), D49.2 (A), D5.2 (A), D50.2 (A), D51.2 (A), D52.2 (A), D53.2 (A), D54.2 (A), D55.2 (A), D56.2 (A), D57.2 (A), D58.2 (A), D59.2 (A), D6.2 (A), D60.2 (A), D61.2 (A), D62.2 (A), D63.2 (A), D64.2 (A), D65.2 (A), D66.2 (A), D67.2 (A), D68.2 (A), D69.2 (A), D7.2 (A), D70.2 (A), D71.2 (A), D72.2 (A), D73.2 (A), D74.2 (A), D75.2 (A), D76.2 (A), D77.2 (A), D78.2 (A), D79.2 (A), D8.2 (A), D80.2 (A), D81.2 (A), D82.2 (A), D83.2 (A), D84.2 (A), D85.2 (A), D86.2 (A), D87.2 (A), D88.2 (A), D89.2 (A), D9.2 (A), D90.2 (A), D91.2 (A), D92.2 (A), D93.2 (A), D94.2 (A), D95.2 (A), D96.2 (A), D97.2 (A), D98.2 (A), D99.2 (A)
- new net: D142.1 (K), D146.1 (K)
- new net: D64.1 (K), D68.1 (K)
- new net: D167.1 (K), D171.1 (K)
- new net: D35.1 (K), D37.1 (K)
- new net: D152.1 (K), D156.1 (K)
- new net: D87.1 (K), D91.1 (K)
- new net: D62.1 (K), D66.1 (K)
- new net: D173.1 (K), D177.1 (K)
- new net: D23.1 (K), D25.1 (K)
- new net: D63.1 (K), D67.1 (K)
- new net: D71.1 (K), D75.1 (K)
- new net: D8.1 (K), D9.1 (K)
- new net: D135.1 (K), D139.1 (K)
- new net: D184.1 (K), D188.1 (K)
- new net: D168.1 (K), D172.1 (K)
- new net: D166.1 (K), D170.1 (K)
- new net: D88.1 (K), D92.1 (K)
- new net: D12.1 (K), D13.1 (K)
- new net: D141.1 (K), D145.1 (K)
- new net: D61.1 (K), D65.1 (K)
- new net: D2.1 (K), D3.1 (K)
- new net: D36.1 (K), D38.1 (K)
- new net: D144.1 (K), D148.1 (K)
- new net: D175.1 (K), D179.1 (K)
- new net: D95.1 (K), D99.1 (K)
- new net: D190.1 (K), D194.1 (K)
- new net: D191.1 (K), D195.1 (K)
- new net: D103.1 (K), D107.1 (K)
- new net: D100.1 (K), D96.1 (K)
- new net: D176.1 (K), D180.1 (K)
- new net: D14.1 (K), D15.1 (K)
- new net: D27.1 (K), D29.1 (K)
- new net: D109.1 (K), D113.1 (K)
- new net: D93.1 (K), D97.1 (K)
- new net: D125.1 (K), D129.1 (K)
- new net: D104.1 (K), D108.1 (K)
- new net: D31.1 (K), D33.1 (K)
- new net: D182.1 (K), D186.1 (K)
- new net: D181.1 (K), D185.1 (K)
- new net: D56.1 (K), D60.1 (K)
- new net: D189.1 (K), D193.1 (K)
- new net: D24.1 (K), D26.1 (K)
- new net: D111.1 (K), D115.1 (K)
- new net: D110.1 (K), D114.1 (K)
- new net: D86.1 (K), D90.1 (K)
- new net: D6.1 (K), D7.1 (K)
- new net: D165.1 (K), D169.1 (K)
- new net: D112.1 (K), D116.1 (K)
- new net: D126.1 (K), D130.1 (K)
- new net: D150.1 (K), D154.1 (K)
- new net: D151.1 (K), D155.1 (K)
- new net: D69.1 (K), D73.1 (K)
- new net: D70.1 (K), D74.1 (K)
- new net: D85.1 (K), D89.1 (K)
- new net: D183.1 (K), D187.1 (K)
- new net: D47.1 (K), D51.1 (K)
- new net: D46.1 (K), D50.1 (K)
- new net: D101.1 (K), D105.1 (K)
- new net: D127.1 (K), D131.1 (K)
- new net: D136.1 (K), D140.1 (K)
- new net: D133.1 (K), D137.1 (K)
- new net: D53.1 (K), D57.1 (K)
- new net: D18.1 (K), D19.1 (K)
- new net: D174.1 (K), D178.1 (K)
- new net: D4.1 (K), D5.1 (K)
- new net: D94.1 (K), D98.1 (K)
- new net: D102.1 (K), D106.1 (K)
- new net: D28.1 (K), D30.1 (K)
- new net: D134.1 (K), D138.1 (K)
- new net: D143.1 (K), D147.1 (K)
- new net: D45.1 (K), D49.1 (K)
- new net: D128.1 (K), D132.1 (K)
- new net: D32.1 (K), D34.1 (K)
- new net: D149.1 (K), D153.1 (K)
- new net: D55.1 (K), D59.1 (K)
- new net: D16.1 (K), D17.1 (K)
- new net: D48.1 (K), D52.1 (K)
- new net: D54.1 (K), D58.1 (K)
- new net: D72.1 (K), D76.1 (K)
- new net: D192.1 (K), D196.1 (K)
Other:
- moved on the sheet: U1, U2

Commit message: hw update for new design
Parts:
- removed D100, D101, D102, D103, D104, D105, D106, D107, D108, D109, D110, D111, D112, D113, D114, D115, D116, D117, D118, D119, D120, D121, D122, D123, D124, D125, D126, D127, D128, D129, D130, D131, D132, D133, D134, D135, D136, D137, D138, D139, D140, D141, D142, D143, D144, D145, D146, D147, D148, D149, D150, D151, D152, D153, D154, D155, D156, D157, D158, D159, D160, D161, D162, D163, D164, D165, D166, D167, D168, D169, D170, D171, D172, D173, D174, D175, D176, D177, D178, D179, D180, D181, D182, D183, D184, D185, D186, D187, D188, D189, D190, D191, D192, D193, D194, D195, D196, D197, D198, D199, D200, D53, D54, D55, D56, D57, D58, D59, D60, D61, D62, D63, D64, D65, D66, D67, D68, D69, D70, D71, D72, D73, D74, D75, D76, D77, D78, D79, D80, D81, D82, D83, D84, D85, D86, D87, D88, D89, D90, D91, D92, D93, D94, D95, D96, D97, D98, D99: LED, Library:LED, symbol Device:LED
- added C1, C2, C4, C5: 33p, symbol Device:C
- added C3, C6, C9: 100n, symbol Device:C_Small
- added C7, C8: 10u, symbol Device:C
- added D53, D54, D55, D56: 3v3, symbol Device:D_Zener
- added R1, R11, R5, R8: 470k, symbol Device:R
- added R10, R2, R4, R7: 0, symbol Device:R
- added R12, R3, R6, R9: 1k, symbol Device:R
- added R13, R14, R15, R16, R17, R18, R20: 100k, symbol Device:R
- added R19: NC, symbol Device:R
- added R21, R22: 1M, symbol Device:R
- added U4: OP_B, Package_SO:SOIC-8_3.9x4.9mm_P1.27mm, symbol Device:Opamp_Dual
- added U5: Opamp_Dual, Package_SO:SOIC-8_3.9x4.9mm_P1.27mm, symbol Device:Opamp_Dual
- D1, D10, D11, D12, D13, D14, D15, D16, D17, D18, D19, D2, D20, D21, D22, D23, D24, D25, D26, D27, D28, D29, D3, D30, D31, D32, D33, D34, D35, D36, D37, D38, D39, D4, D40, D41, D42, D43, D44, D45, D46, D47, D48, D49, D5, D50, D51, D52, D6, D7, D8, D9: footprint Library:LED -> LED_THT:LED_D5.0mm_Clear
- U3: value Opamp_Dual -> OP_T
Connections:
- net GND: now also U3.4 (V-), C3.2, C6.2, C7.2, C8.2, C9.2, R10.1, R14.1, R19.2, R2.1, R22.2, R4.1, R7.1, U4.4 (V-), U5.4 (V-)
- net ARR_BR: now reaches D35.1 (K), D37.1 (K)
- net ARR_BR: now also D27.1 (K), D28.1 (K), D29.1 (K), D30.1 (K), D31.1 (K), D32.1 (K), D33.1 (K), D34.1 (K), D36.1 (K), D38.1 (K), D39.1 (K), C5.1, D56.2 (A), R11.1, R15.1, U4.5 (+)
- net ARR_TR: now reaches D23.1 (K), D25.1 (K)
- net ARR_TR: now also D14.1 (K), D15.1 (K), D16.1 (K), D17.1 (K), D18.1 (K), D19.1 (K), D20.1 (K), D21.1 (K), D22.1 (K), D24.1 (K), D26.1 (K), U3.5 (+), C2.1, D54.2 (A), R17.1, R5.1
- net ARR_TL: now reaches D8.1 (K), D9.1 (K)
- net ARR_TL: now also D1.1 (K), D10.1 (K), D11.1 (K), D12.1 (K), D13.1 (K), D2.1 (K), D3.1 (K), D4.1 (K), D5.1 (K), D6.1 (K), D7.1 (K), U3.2 (-), C1.1, D53.2 (A), R1.1, R18.1
- net ARR_BL: now reaches D42.1 (K)
- net ARR_BL: now also D40.1 (K), D41.1 (K), D43.1 (K), D44.1 (K), D45.1 (K), D46.1 (K), D47.1 (K), D48.1 (K), D49.1 (K), D50.1 (K), D51.1 (K), D52.1 (K), C4.1, D55.2 (A), R16.1, R8.1, U4.2 (-)
- net VCC: now reaches U3.8 (V+)
- net VCC: now also C3.1, C6.1, C9.1, U4.8 (V+), U5.8 (V+)
- net at U3.6 (-): now also R4.2
- net at U3.7: now also C2.2, R5.2, R6.2
- net at U3.1: now also C1.2, R1.2, R3.2
- net at U3.3 (+): now also R2.2
- new net: R7.2, U4.3 (+)
- new net: R15.2, R16.2, R17.2, R18.2, R19.1, U5.3 (+)
- new net: R10.2, U4.6 (-)
- new net: R13.1, R14.2, U5.2 (-)
- new net: R13.2, R20.1, U5.1, U5.5 (+)
- new net: D55.1 (K), R9.1
- new net: C4.2, R8.2, R9.2, U4.1
- new net: R21.2, R22.1, U5.6 (-)
- new net: C7.1, C8.1, R20.2, R21.1
- new net: D53.1 (K), R3.1
- new net: C5.2, R11.2, R12.2, U4.7
- new net: D56.1 (K), R12.1
- new net: D54.1 (K), R6.1
- new net OUT: U5.7
Other:
- moved on the sheet: U1, U3A, U3B, U3C

Commit message: sch finished
Parts:
- removed U1: TP4056-42-ESOP8, Package_SO:SOIC-8-1EP_3.9x4.9mm_P1.27mm_EP2.41x3.3mm_ThermalVias, symbol Battery_Management:TP4056-42-ESOP8
- added C10, C11, C12: 100n, Capacitor_SMD:C_0603_1608Metric, symbol Device:C_Small
- added C13, C15: 10u, Capacitor_SMD:C_0603_1608Metric, symbol Device:C
- added C14, C16, C20, C22: 100n, Capacitor_SMD:C_0603_1608Metric, symbol Device:C
- added C17, C18: 1u, Capacitor_SMD:C_0603_1608Metric, symbol Device:C_Small
- added C19, C21, C24: 4u7, Capacitor_SMD:C_0603_1608Metric, symbol Device:C
- added C23: 2u2, Capacitor_SMD:C_0603_1608Metric, symbol Device:C
- added D57: LED, LED_SMD:LED_0805_2012Metric, symbol Device:LED
- added D58, D59, D60, D61: LED, Capacitor_SMD:C_0603_1608Metric, symbol Device:LED
- added DS1: OLED-128O032D, Library:OLED-128O032D, symbol Library:OLED-128O032D
- added J1: DBG, Connector_PinHeader_2.54mm:PinHeader_1x08_P2.54mm_Vertical, symbol Connector:Conn_01x08_Pin
- added J2: BAT, Connector_JST:JST_XH_B2B-XH-A_1x02_P2.50mm_Vertical, symbol Connector:Conn_01x02_Socket
- added R23, R24, R25: 10k, Resistor_SMD:R_0603_1608Metric, symbol Device:R
- added R26: 560k, Resistor_SMD:R_0603_1608Metric, symbol Device:R
- added R27, R28, R29: 4k7, Resistor_SMD:R_0603_1608Metric, symbol Device:R
- added RV1, RV2, RV3, RV4: 2k, Potentiometer_SMD:Potentiometer_Bourns_TC33X_Vertical, symbol Device:R_Potentiometer
- added SW1: BUTTON, Button_Switch_SMD:SW_Push_1P1T_NO_Vertical_Wuerth_434133025816, symbol Switch:SW_Push
- added SW2: RESET, Button_Switch_SMD:SW_Push_1P1T_NO_Vertical_Wuerth_434133025816, symbol Switch:SW_Push
- added U1: TLV75733PDBV, Package_TO_SOT_SMD:SOT-23-5, symbol Regulator_Linear:TLV75733PDBV
- C1, C2, C3, C4, C5, C6, C7, C8, C9: footprint (none) -> Capacitor_SMD:C_0603_1608Metric
- D1: footprint LED_THT:LED_D5.0mm_Clear -> Capacitor_SMD:C_0603_1608Metric
- D53, D54, D55, D56: footprint (none) -> Diode_SMD:D_SOD-123
- R1, R10, R11, R12, R13, R14, R15, R16, R17, R18, R19, R2, R20, R21, R22, R3, R4, R5, R6, R7, R8, R9: footprint (none) -> Resistor_SMD:R_0603_1608Metric
Connections:
- net GND: now also U2.4 (VSS), C10.2, C11.2, C12.2, C13.2, C14.2, C15.2, C16.2, C19.2, C20.2, C21.2, C22.2, C23.2, C24.2, D58.1 (K), D59.1 (K), D60.1 (K), D61.1 (K), DS1.7 (VSS), J1.8 (Pin_8), J2.2 (Pin_2), R26.1, SW1.2, SW2.2, U1.2 (GND)
- net OUT: now also U2.9 (PA3)
- net VCC: now also C15.1, C16.1, J1.1 (Pin_1), J2.1 (Pin_1), U1.1 (IN), U1.3 (EN)
- net ADC_IN0: now reaches R13.2, R20.1, U5.1, U5.5 (+)
- net ADC_IN0: now also U2.6 (PA0)
- net ~{RES}: now reaches U2.17 (PC6)
- net ~{RES}: now also C24.1, DS1.9 (~{RES}), R29.1
- net SCL: now reaches U2.18 (PA9/PA11)
- net SCL: now also DS1.10 (SCL), R28.2
- net SDA: now reaches U2.19 (PA10/PA12)
- net SDA: now also DS1.11 (SDA), R27.2
- net SWDIO: now reaches U2.20 (PA13)
- net SWDIO: now also J1.4 (Pin_4)
- net SWCLK: now reaches U2.21 (PA14)
- net SWCLK: now also J1.3 (Pin_3)
- net at U2.22 (PA15): now also D57.1 (K)
- net U1TXD: now reaches U2.26 (PB6)
- net U1TXD: now also J1.5 (Pin_5)
- net U1RXD: now reaches U2.27 (PB7)
- net U1RXD: now also J1.6 (Pin_6)
- net +3V3: now reaches U2.3 (VDD)
- net +3V3: now also C12.1, C13.1, C14.1, C21.1, C22.1, DS1.5 (VBAT), DS1.8 (VDD), J1.2 (Pin_2), R23.1, R24.1, R25.1, R27.1, R28.1, R29.2, RV1.1, RV1.2, RV2.1, RV2.2, RV3.1, RV3.2, RV4.1, RV4.2, U1.5 (OUT)
- net ~{RESET}: now reaches U2.5 (PF2)
- net ~{RESET}: now also C10.1, J1.7 (Pin_7), R23.2, SW2.1
- net BUTTON: now reaches U2.7 (PA1)
- net BUTTON: now also C11.1, R24.2, SW1.1
- new net: D59.2 (A), RV2.3
- new net: C19.1, C20.1, DS1.14 (VCC)
- new net: D61.2 (A), RV4.3
- new net: D57.2 (A), R25.2
- new net: C23.1, DS1.13 (VCOMH)
- new net: D58.2 (A), RV1.3
- new net: DS1.12 (IREF), R26.2
- new net: C18.1, DS1.4 (C1N)
- new net: C18.2, DS1.3 (C1P)
- new net: C17.2, DS1.1 (C2N)
- new net: C17.1, DS1.2 (C2P)
- new net: D60.2 (A), RV3.3
- no-connect marks 0 -> 15
Other:
- moved on the sheet: U2

Commit message: hw pcb init
Parts:
- removed D1, D59, D60, D61: LED, Capacitor_SMD:C_0603_1608Metric, symbol Device:LED
- removed D10, D14, D15, D16, D19, D2, D23, D27, D28, D29, D3, D32, D40, D41, D42, D45, D49, D6: LED, LED_THT:LED_D5.0mm_Clear, symbol Device:LED
- added D34, D35: LED, LED_THT:LED_D5.0mm_Clear, symbol Device:LED
- added H1, H2, H3, H4: MountingHole_Pad, MountingHole:MountingHole_3.2mm_M3_Pad, symbol Mechanical:MountingHole_Pad
- D33: renamed from D58; footprint Capacitor_SMD:C_0603_1608Metric -> LED_THT:LED_D5.0mm_Clear
- renumbered D4 to D1, D17 to D10, D26 to D14, D22 to D15, D18 to D16, D44 to D17, D48 to D18, D52 to D19, D5 to D2, D39 to D20, D35 to D21, D31 to D22, D43 to D23, D47 to D24, D51 to D25, D38 to D26, D34 to D27, D30 to D28, D46 to D29, D24 to D3, D50 to D30, D37 to D31, D33 to D32, D53 to D37, D54 to D38, D55 to D39, D20 to D4, D56 to D40, D57 to D41, D7 to D5, D8 to D6, D9 to D7, D25 to D8, D21 to D9
Connections:
- net ARR_BL: now also U4.5 (+); no longer U4.2 (-)
- net ARR_BR: now also U4.2 (-); no longer D36.1 (K), U4.5 (+)
- net GND: now also D36.1 (K), D34.1 (K), D35.1 (K), H1.1, H2.1, H3.1, H4.1; no longer D36.2 (A)
- net at RV2.3: now also D34.2 (A)
- net at R7.2: now also U4.6 (-); no longer U4.3 (+)
- net at R10.2: now also U4.3 (+); no longer U4.6 (-)
- net at RV4.3: now also D36.2 (A)
- net at C4.2, R8.2, R9.2: now also U4.7; no longer U4.1
- net at C5.2, R11.2, R12.2: now also U4.1; no longer U4.7
- net at RV3.3: now also D35.2 (A)

Commit message: hw ver1
Parts:
- added C25, C26: 10u, Capacitor_SMD:C_0603_1608Metric, symbol Device:C
- added C27: 100n, Capacitor_SMD:C_0603_1608Metric, symbol Device:C
- added J3: USB_C_Receptacle_PowerOnly_6P, Connector_USB:USB_C_Receptacle_GCT_USB4125-xx-x_6P_TopMnt_Horizontal, symbol Connector:USB_C_Receptacle_PowerOnly_6P
- added R30, R31, R32: 5k1, Resistor_SMD:R_0603_1608Metric, symbol Device:R
- added U6: TP4056-42-ESOP8, Package_SO:SOIC-8-1EP_3.9x4.9mm_P1.27mm_EP2.41x3.3mm, symbol Battery_Management:TP4056-42-ESOP8
Connections:
- net ARR_BL: now also U4.6 (-); no longer R16.1, U4.5 (+)
- net ARR_BR: no longer R15.1
- net ARR_TL: no longer R18.1
- net ARR_TR: now also U3.6 (-); no longer R17.1, U3.5 (+)
- net GND: now also J1.3 (Pin_3), C25.2, C26.2, C27.2, J3.A12 (GND), J3.B12 (GND), J3.S1 (SHIELD), R30.2, R31.2, R32.2, U6.1 (TEMP), U6.3 (GND), U6.9 (EPAD); no longer J1.8 (Pin_8)
- net SWCLK: now also J1.5 (Pin_5); no longer J1.3 (Pin_3)
- net U1RXD: now also J1.7 (Pin_7); no longer J1.6 (Pin_6)
- net U1TXD: now also J1.6 (Pin_6); no longer J1.5 (Pin_5)
- net VCC: now also C26.1, C27.1, U6.5 (BAT)
- net ~{RESET}: now also J1.8 (Pin_8); no longer J1.7 (Pin_7)
- net at R7.2: now also U4.5 (+); no longer U4.6 (-)
- net O3: now reaches C4.2, R8.2, R9.2, U4.7
- net O3: now also R16.1
- net O4: now reaches C5.2, R11.2, R12.2, U4.1
- net O4: now also R15.1
- net O1: now reaches C1.2, R1.2, R3.2, U3.1
- net O1: now also R18.1
- net O2: now reaches C2.2, R5.2, R6.2, U3.7
- net O2: now also R17.1
- net at R4.2: now also U3.5 (+); no longer U3.6 (-)
- new net: J3.A5 (CC1), R30.1
- new net: J3.B5 (CC2), R31.1
- new net: R32.1, U6.2 (PROG)
- new net VBUS: C25.1, J3.A9 (VBUS), J3.B9 (VBUS), U6.4 (V_{CC}), U6.8 (CE)
- no-connect marks 15 -> 17
Other:
- moved on the sheet: C13, C14, C15, C16, D33, D34, D35, D36, H1, H2, H3, H4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

Commit message: hw rev2
Parts:
- added R33, R34: 10k, Resistor_SMD:R_0603_1608Metric, symbol Device:R
Connections:
- net ADC_IN0: now also R33.1; no longer U2.6 (PA0)
- net GND: now also R34.2
- new net: R33.2, R34.1, U2.6 (PA0)
